Commit message: Path planning added

File: urdf/arm.xacro (robot description, xacro)
@@ -5,5 +5,5 @@
 <xacro:include filename="$(find main_description)/urdf/Design.trans" />
 <!--  PROPERTIES  -->
-<xacro:property name="strength" value="2000"/>
+<xacro:property name="strength" value="1000"/>
 <xacro:property name="speed" value = "0.01"/>
 <xacro:property name="damping" value = "0"/>

File: urdf/description_log.urdf (robot description, URDF)
Before this commit: robot Design, 54 links, 53 joints
Joints:
- joint Joint2: limit lower=-1.570796 upper=1.570796 effort=2000 velocity=0.01 -> lower=-1.570796 upper=1.570796 effort=1000 velocity=0.01
- joint Joint3: limit lower=-1.570796 upper=1.570796 effort=2000 velocity=0.01 -> lower=-1.570796 upper=1.570796 effort=1000 velocity=0.01
- joint anchor: limit lower=0 upper=6.28318 effort=2000 velocity=1 -> lower=0 upper=6.28318 effort=1000 velocity=1
- joint base_link: limit lower=-3.04 upper=-0.1 effort=2000 velocity=0.01 -> lower=-3.04 upper=-0.1 effort=1000 velocity=0.01

Commit message: Coordinate input working

File: urdf/arm.xacro (robot description, xacro)
@@ -12,5 +12,5 @@
 <joint name="anchor" type="continuous">
   <axis xyz="0 0 1"/>
-	<origin xyz="0.0 0.0 0.02" rpy="0 0 0" />
+	<origin xyz="0.0 0.0 0.1" rpy="0 0 0" />
 	<parent link="world"/>
 	<child link="base_link"/>

File: urdf/description_log.urdf (robot description, URDF)
Before this commit: robot Design, 54 links, 53 joints
Joints:
- joint LBseg10_LBseg11_joint: origin xyz=0 0 0.0125 rpy=0 0 0 -> xyz=0 0 0.0175 rpy=0 0 0
- joint LBseg11_LBseg12_joint: origin xyz=0 0 0.0125 rpy=0 0 0 -> xyz=0 0 0.0175 rpy=0 0 0
- joint LBseg1_LBseg2_joint: origin xyz=0 0 0.0125 rpy=0 0 0 -> xyz=0 0 0.0175 rpy=0 0 0
- joint LBseg2_LBseg3_joint: origin xyz=0 0 0.0125 rpy=0 0 0 -> xyz=0 0 0.0175 rpy=0 0 0
- joint LBseg3_LBseg4_joint: origin xyz=0 0 0.0125 rpy=0 0 0 -> xyz=0 0 0.0175 rpy=0 0 0
- joint LBseg4_LBseg5_joint: origin xyz=0 0 0.0125 rpy=0 0 0 -> xyz=0 0 0.0175 rpy=0 0 0
- joint LBseg5_LBseg6_joint: origin xyz=0 0 0.0125 rpy=0 0 0 -> xyz=0 0 0.0175 rpy=0 0 0
- joint LBseg6_LBseg7_joint: origin xyz=0 0 0.0125 rpy=0 0 0 -> xyz=0 0 0.0175 rpy=0 0 0
- joint LBseg7_LBseg8_joint: origin xyz=0 0 0.0125 rpy=0 0 0 -> xyz=0 0 0.0175 rpy=0 0 0
- joint LBseg8_LBseg9_joint: origin xyz=0 0 0.0125 rpy=0 0 0 -> xyz=0 0 0.0175 rpy=0 0 0
- joint LBseg9_LBseg10_joint: origin xyz=0 0 0.0125 rpy=0 0 0 -> xyz=0 0 0.0175 rpy=0 0 0
- joint LTseg10_LTseg11_joint: origin xyz=0 0 0.0125 rpy=0 0 0 -> xyz=0 0 0.0175 rpy=0 0 0
- joint LTseg11_LTseg12_joint: origin xyz=0 0 0.0125 rpy=0 0 0 -> xyz=0 0 0.0175 rpy=0 0 0
- joint LTseg1_LTseg2_joint: origin xyz=0 0 0.0125 rpy=0 0 0 -> xyz=0 0 0.0175 rpy=0 0 0
- joint LTseg2_LTseg3_joint: origin xyz=0 0 0.0125 rpy=0 0 0 -> xyz=0 0 0.0175 rpy=0 0 0
- joint LTseg3_LTseg4_joint: origin xyz=0 0 0.0125 rpy=0 0 0 -> xyz=0 0 0.0175 rpy=0 0 0
- joint LTseg4_LTseg5_joint: origin xyz=0 0 0.0125 rpy=0 0 0 -> xyz=0 0 0.0175 rpy=0 0 0
- joint LTseg5_LTseg6_joint: origin xyz=0 0 0.0125 rpy=0 0 0 -> xyz=0 0 0.0175 rpy=0 0 0
- joint LTseg6_LTseg7_joint: origin xyz=0 0 0.0125 rpy=0 0 0 -> xyz=0 0 0.0175 rpy=0 0 0
- joint LTseg7_LTseg8_joint: origin xyz=0 0 0.0125 rpy=0 0 0 -> xyz=0 0 0.0175 rpy=0 0 0
- joint LTseg8_LTseg9_joint: origin xyz=0 0 0.0125 rpy=0 0 0 -> xyz=0 0 0.0175 rpy=0 0 0
- joint LTseg9_LTseg10_joint: origin xyz=0 0 0.0125 rpy=0 0 0 -> xyz=0 0 0.0175 rpy=0 0 0
- joint RBseg10_RBseg11_joint: origin xyz=0 0 0.0125 rpy=0 0 0 -> xyz=0 0 0.0175 rpy=0 0 0
- joint RBseg11_RBseg12_joint: origin xyz=0 0 0.0125 rpy=0 0 0 -> xyz=0 0 0.0175 rpy=0 0 0
- joint RBseg1_RBseg2_joint: origin xyz=0 0 0.0125 rpy=0 0 0 -> xyz=0 0 0.0175 rpy=0 0 0
- joint RBseg2_RBseg3_joint: origin xyz=0 0 0.0125 rpy=0 0 0 -> xyz=0 0 0.0175 rpy=0 0 0
- joint RBseg3_RBseg4_joint: origin xyz=0 0 0.0125 rpy=0 0 0 -> xyz=0 0 0.0175 rpy=0 0 0
- joint RBseg4_RBseg5_joint: origin xyz=0 0 0.0125 rpy=0 0 0 -> xyz=0 0 0.0175 rpy=0 0 0
- joint RBseg5_RBseg6_joint: origin xyz=0 0 0.0125 rpy=0 0 0 -> xyz=0 0 0.0175 rpy=0 0 0
- joint RBseg6_RBseg7_joint: origin xyz=0 0 0.0125 rpy=0 0 0 -> xyz=0 0 0.0175 rpy=0 0 0
- joint RBseg7_RBseg8_joint: origin xyz=0 0 0.0125 rpy=0 0 0 -> xyz=0 0 0.0175 rpy=0 0 0
- joint RBseg8_RBseg9_joint: origin xyz=0 0 0.0125 rpy=0 0 0 -> xyz=0 0 0.0175 rpy=0 0 0
- joint RBseg9_RBseg10_joint: origin xyz=0 0 0.0125 rpy=0 0 0 -> xyz=0 0 0.0175 rpy=0 0 0
- joint RTseg10_RTseg11_joint: origin xyz=0 0 0.0125 rpy=0 0 0 -> xyz=0 0 0.0175 rpy=0 0 0
- joint RTseg11_RTseg12_joint: origin xyz=0 0 0.0125 rpy=0 0 0 -> xyz=0 0 0.0175 rpy=0 0 0
- joint RTseg1_RTseg2_joint: origin xyz=0 0 0.0125 rpy=0 0 0 -> xyz=0 0 0.0175 rpy=0 0 0
- joint RTseg2_RTseg3_joint: origin xyz=0 0 0.0125 rpy=0 0 0 -> xyz=0 0 0.0175 rpy=0 0 0
- joint RTseg3_RTseg4_joint: origin xyz=0 0 0.0125 rpy=0 0 0 -> xyz=0 0 0.0175 rpy=0 0 0
- joint RTseg4_RTseg5_joint: origin xyz=0 0 0.0125 rpy=0 0 0 -> xyz=0 0 0.0175 rpy=0 0 0
- joint RTseg5_RTseg6_joint: origin xyz=0 0 0.0125 rpy=0 0 0 -> xyz=0 0 0.0175 rpy=0 0 0
- joint RTseg6_RTseg7_joint: origin xyz=0 0 0.0125 rpy=0 0 0 -> xyz=0 0 0.0175 rpy=0 0 0
- joint RTseg7_RTseg8_joint: origin xyz=0 0 0.0125 rpy=0 0 0 -> xyz=0 0 0.0175 rpy=0 0 0
- joint RTseg8_RTseg9_joint: origin xyz=0 0 0.0125 rpy=0 0 0 -> xyz=0 0 0.0175 rpy=0 0 0
- joint RTseg9_RTseg10_joint: origin xyz=0 0 0.0125 rpy=0 0 0 -> xyz=0 0 0.0175 rpy=0 0 0
- joint anchor: origin xyz=0.0 0.0 0.02 rpy=0 0 0 -> xyz=0.0 0.0 0.1 rpy=0 0 0

File: urdf/macros2.xacro (robot description, xacro)
@@ -47,5 +47,5 @@
 		<limit effort="${fingerForce}" lower="-0.25" upper="0.25" velocity="0.001"/>
 		<dynamics damping="0.05" friction="0.0"/>
-		<origin xyz="0 0 ${length}" rpy="0 0 0"/>
+		<origin xyz="0 0 ${length+0.005}" rpy="0 0 0"/>
 		<parent link="${seg1}"/>
 		<child link="${seg2}"/>
@@ -59,4 +59,5 @@
 		<axis xyz="1 0 0"/>
 		<limit effort="${fingerForce}" lower="-0.1" upper="0.1" velocity="0.0001"/>
+		<!--<dynamics damping="0.05" friction="0.0"/>-->
 		<origin xyz="${offset}" rpy="${rotation}"/>
 		<parent link="${seg1}"/>

Commit message: New model, controller complete
Model added, path finding, speed control for constant effector angle and PID values

File: urdf/arm.xacro (robot description, xacro)
@@ -125,5 +125,5 @@
   <child link="Link1_1"/>
   <axis xyz="0.0 0.0 1.0"/>
-  <limit effort="${strength}" lower="0.0" upper="6.283185" velocity="${speed}"/>
+  <limit effort="${strength}" lower="-6.283185" upper="6.283185" velocity="${speed}"/>
   <dynamics damping="${damping}" friction="0.0"/>
 </joint>

File: urdf/description_log.urdf (robot description, URDF)
Before this commit: robot Design, 55 links, 54 joints
Joints:
- joint Rev1: limit lower=0.0 upper=6.283185 effort=1000 velocity=0.01 -> lower=-6.283185 upper=6.283185 effort=1000 velocity=0.01
