Commit message: Gripper position estimation
rough estimation from stess/strain sensors

File: urdf/description_log.urdf (robot description, URDF)
Before this commit: robot Design, 55 links, 54 joints
Links:
- link LBseg10: geometry collision box size=0.0125 0.0125 0.0125; visual box size=0.0125 0.0125 0.0125
- link LBseg11: geometry collision box size=0.0116666666667 0.0116666666667 0.0125; visual box size=0.0116666666667 0.0116666666667 0.0125
- link LBseg12: geometry collision box size=0.0108333333333 0.0108333333333 0.0125; visual box size=0.0108333333333 0.0108333333333 0.0125
- link LBseg2: geometry collision box size=0.0191666666667 0.0191666666667 0.0125; visual box size=0.0191666666667 0.0191666666667 0.0125
- link LBseg3: geometry collision box size=0.0183333333333 0.0183333333333 0.0125; visual box size=0.0183333333333 0.0183333333333 0.0125
- link LBseg4: geometry collision box size=0.0175 0.0175 0.0125; visual box size=0.0175 0.0175 0.0125
- link LBseg5: geometry collision box size=0.0166666666667 0.0166666666667 0.0125; visual box size=0.0166666666667 0.0166666666667 0.0125
- link LBseg6: geometry collision box size=0.0158333333333 0.0158333333333 0.0125; visual box size=0.0158333333333 0.0158333333333 0.0125
- link LBseg7: geometry collision box size=0.015 0.015 0.0125; visual box size=0.015 0.015 0.0125
- link LBseg8: geometry collision box size=0.0141666666667 0.0141666666667 0.0125; visual box size=0.0141666666667 0.0141666666667 0.0125
- link LBseg9: geometry collision box size=0.0133333333333 0.0133333333333 0.0125; visual box size=0.0133333333333 0.0133333333333 0.0125
- link LTseg10: geometry collision box size=0.0125 0.0125 0.0125; visual box size=0.0125 0.0125 0.0125
- link LTseg11: geometry collision box size=0.0116666666667 0.0116666666667 0.0125; visual box size=0.0116666666667 0.0116666666667 0.0125
- link LTseg12: geometry collision box size=0.0108333333333 0.0108333333333 0.0125; visual box size=0.0108333333333 0.0108333333333 0.0125
- link LTseg2: geometry collision box size=0.0191666666667 0.0191666666667 0.0125; visual box size=0.0191666666667 0.0191666666667 0.0125
- link LTseg3: geometry collision box size=0.0183333333333 0.0183333333333 0.0125; visual box size=0.0183333333333 0.0183333333333 0.0125
- link LTseg4: geometry collision box size=0.0175 0.0175 0.0125; visual box size=0.0175 0.0175 0.0125
- link LTseg5: geometry collision box size=0.0166666666667 0.0166666666667 0.0125; visual box size=0.0166666666667 0.0166666666667 0.0125
- link LTseg6: geometry collision box size=0.0158333333333 0.0158333333333 0.0125; visual box size=0.0158333333333 0.0158333333333 0.0125
- link LTseg7: geometry collision box size=0.015 0.015 0.0125; visual box size=0.015 0.015 0.0125
- link LTseg8: geometry collision box size=0.0141666666667 0.0141666666667 0.0125; visual box size=0.0141666666667 0.0141666666667 0.0125
- link LTseg9: geometry collision box size=0.0133333333333 0.0133333333333 0.0125; visual box size=0.0133333333333 0.0133333333333 0.0125
- link RBseg10: geometry collision box size=0.0125 0.0125 0.0125; visual box size=0.0125 0.0125 0.0125
- link RBseg11: geometry collision box size=0.0116666666667 0.0116666666667 0.0125; visual box size=0.0116666666667 0.0116666666667 0.0125
- link RBseg12: geometry collision box size=0.0108333333333 0.0108333333333 0.0125; visual box size=0.0108333333333 0.0108333333333 0.0125
- link RBseg2: geometry collision box size=0.0191666666667 0.0191666666667 0.0125; visual box size=0.0191666666667 0.0191666666667 0.0125
- link RBseg3: geometry collision box size=0.0183333333333 0.0183333333333 0.0125; visual box size=0.0183333333333 0.0183333333333 0.0125
- link RBseg4: geometry collision box size=0.0175 0.0175 0.0125; visual box size=0.0175 0.0175 0.0125
- link RBseg5: geometry collision box size=0.0166666666667 0.0166666666667 0.0125; visual box size=0.0166666666667 0.0166666666667 0.0125
- link RBseg6: geometry collision box size=0.0158333333333 0.0158333333333 0.0125; visual box size=0.0158333333333 0.0158333333333 0.0125
- link RBseg7: geometry collision box size=0.015 0.015 0.0125; visual box size=0.015 0.015 0.0125
- link RBseg8: geometry collision box size=0.0141666666667 0.0141666666667 0.0125; visual box size=0.0141666666667 0.0141666666667 0.0125
- link RBseg9: geometry collision box size=0.0133333333333 0.0133333333333 0.0125; visual box size=0.0133333333333 0.0133333333333 0.0125
- link RTseg10: geometry collision box size=0.0125 0.0125 0.0125; visual box size=0.0125 0.0125 0.0125
- link RTseg11: geometry collision box size=0.0116666666667 0.0116666666667 0.0125; visual box size=0.0116666666667 0.0116666666667 0.0125
- link RTseg12: geometry collision box size=0.0108333333333 0.0108333333333 0.0125; visual box size=0.0108333333333 0.0108333333333 0.0125
- link RTseg2: geometry collision box size=0.0191666666667 0.0191666666667 0.0125; visual box size=0.0191666666667 0.0191666666667 0.0125
- link RTseg3: geometry collision box size=0.0183333333333 0.0183333333333 0.0125; visual box size=0.0183333333333 0.0183333333333 0.0125
- link RTseg4: geometry collision box size=0.0175 0.0175 0.0125; visual box size=0.0175 0.0175 0.0125
- link RTseg5: geometry collision box size=0.0166666666667 0.0166666666667 0.0125; visual box size=0.0166666666667 0.0166666666667 0.0125
- link RTseg6: geometry collision box size=0.0158333333333 0.0158333333333 0.0125; visual box size=0.0158333333333 0.0158333333333 0.0125
- link RTseg7: geometry collision box size=0.015 0.015 0.0125; visual box size=0.015 0.015 0.0125
- link RTseg8: geometry collision box size=0.0141666666667 0.0141666666667 0.0125; visual box size=0.0141666666667 0.0141666666667 0.0125
- link RTseg9: geometry collision box size=0.0133333333333 0.0133333333333 0.0125; visual box size=0.0133333333333 0.0133333333333 0.0125
Joints:
- joint LBseg10_LBseg11_joint: limit lower=-0.25 upper=0.25 effort=1 velocity=0.001 -> lower=-0.25 upper=0.25 effort=0.680555555556 velocity=0.001
- joint LBseg11_LBseg12_joint: limit lower=-0.25 upper=0.25 effort=1 velocity=0.001 -> lower=-0.25 upper=0.25 effort=0.586805555556 velocity=0.001
- joint LBseg1_LBseg2_joint: limit lower=-0.25 upper=0.25 effort=1 velocity=0.001 -> lower=-0.25 upper=0.25 effort=1.83680555556 velocity=0.001
- joint LBseg2_LBseg3_joint: limit lower=-0.25 upper=0.25 effort=1 velocity=0.001 -> lower=-0.25 upper=0.25 effort=1.68055555556 velocity=0.001
- joint LBseg3_LBseg4_joint: limit lower=-0.25 upper=0.25 effort=1 velocity=0.001 -> lower=-0.25 upper=0.25 effort=1.53125 velocity=0.001
- joint LBseg4_LBseg5_joint: limit lower=-0.25 upper=0.25 effort=1 velocity=0.001 -> lower=-0.25 upper=0.25 effort=1.38888888889 velocity=0.001
- joint LBseg5_LBseg6_joint: limit lower=-0.25 upper=0.25 effort=1 velocity=0.001 -> lower=-0.25 upper=0.25 effort=1.25347222222 velocity=0.001
- joint LBseg6_LBseg7_joint: limit lower=-0.25 upper=0.25 effort=1 velocity=0.001 -> lower=-0.25 upper=0.25 effort=1.125 velocity=0.001
- joint LBseg7_LBseg8_joint: limit lower=-0.25 upper=0.25 effort=1 velocity=0.001 -> lower=-0.25 upper=0.25 effort=1.00347222222 velocity=0.001
- joint LBseg8_LBseg9_joint: limit lower=-0.25 upper=0.25 effort=1 velocity=0.001 -> lower=-0.25 upper=0.25 effort=0.888888888889 velocity=0.001
- joint LBseg9_LBseg10_joint: limit lower=-0.25 upper=0.25 effort=1 velocity=0.001 -> lower=-0.25 upper=0.25 effort=0.78125 velocity=0.001
- joint LTseg10_LTseg11_joint: limit lower=-0.25 upper=0.25 effort=1 velocity=0.001 -> lower=-0.25 upper=0.25 effort=0.680555555556 velocity=0.001
- joint LTseg11_LTseg12_joint: limit lower=-0.25 upper=0.25 effort=1 velocity=0.001 -> lower=-0.25 upper=0.25 effort=0.586805555556 velocity=0.001
- joint LTseg1_LTseg2_joint: limit lower=-0.25 upper=0.25 effort=1 velocity=0.001 -> lower=-0.25 upper=0.25 effort=1.83680555556 velocity=0.001
- joint LTseg2_LTseg3_joint: limit lower=-0.25 upper=0.25 effort=1 velocity=0.001 -> lower=-0.25 upper=0.25 effort=1.68055555556 velocity=0.001
- joint LTseg3_LTseg4_joint: limit lower=-0.25 upper=0.25 effort=1 velocity=0.001 -> lower=-0.25 upper=0.25 effort=1.53125 velocity=0.001
- joint LTseg4_LTseg5_joint: limit lower=-0.25 upper=0.25 effort=1 velocity=0.001 -> lower=-0.25 upper=0.25 effort=1.38888888889 velocity=0.001
- joint LTseg5_LTseg6_joint: limit lower=-0.25 upper=0.25 effort=1 velocity=0.001 -> lower=-0.25 upper=0.25 effort=1.25347222222 velocity=0.001
- joint LTseg6_LTseg7_joint: limit lower=-0.25 upper=0.25 effort=1 velocity=0.001 -> lower=-0.25 upper=0.25 effort=1.125 velocity=0.001
- joint LTseg7_LTseg8_joint: limit lower=-0.25 upper=0.25 effort=1 velocity=0.001 -> lower=-0.25 upper=0.25 effort=1.00347222222 velocity=0.001
- joint LTseg8_LTseg9_joint: limit lower=-0.25 upper=0.25 effort=1 velocity=0.001 -> lower=-0.25 upper=0.25 effort=0.888888888889 velocity=0.001
- joint LTseg9_LTseg10_joint: limit lower=-0.25 upper=0.25 effort=1 velocity=0.001 -> lower=-0.25 upper=0.25 effort=0.78125 velocity=0.001
- joint RBseg10_RBseg11_joint: limit lower=-0.25 upper=0.25 effort=1 velocity=0.001 -> lower=-0.25 upper=0.25 effort=0.680555555556 velocity=0.001
- joint RBseg11_RBseg12_joint: limit lower=-0.25 upper=0.25 effort=1 velocity=0.001 -> lower=-0.25 upper=0.25 effort=0.586805555556 velocity=0.001
- joint RBseg1_RBseg2_joint: limit lower=-0.25 upper=0.25 effort=1 velocity=0.001 -> lower=-0.25 upper=0.25 effort=1.83680555556 velocity=0.001
- joint RBseg2_RBseg3_joint: limit lower=-0.25 upper=0.25 effort=1 velocity=0.001 -> lower=-0.25 upper=0.25 effort=1.68055555556 velocity=0.001
- joint RBseg3_RBseg4_joint: limit lower=-0.25 upper=0.25 effort=1 velocity=0.001 -> lower=-0.25 upper=0.25 effort=1.53125 velocity=0.001
- joint RBseg4_RBseg5_joint: limit lower=-0.25 upper=0.25 effort=1 velocity=0.001 -> lower=-0.25 upper=0.25 effort=1.38888888889 velocity=0.001
- joint RBseg5_RBseg6_joint: limit lower=-0.25 upper=0.25 effort=1 velocity=0.001 -> lower=-0.25 upper=0.25 effort=1.25347222222 velocity=0.001
- joint RBseg6_RBseg7_joint: limit lower=-0.25 upper=0.25 effort=1 velocity=0.001 -> lower=-0.25 upper=0.25 effort=1.125 velocity=0.001
- joint RBseg7_RBseg8_joint: limit lower=-0.25 upper=0.25 effort=1 velocity=0.001 -> lower=-0.25 upper=0.25 effort=1.00347222222 velocity=0.001
- joint RBseg8_RBseg9_joint: limit lower=-0.25 upper=0.25 effort=1 velocity=0.001 -> lower=-0.25 upper=0.25 effort=0.888888888889 velocity=0.001
- joint RBseg9_RBseg10_joint: limit lower=-0.25 upper=0.25 effort=1 velocity=0.001 -> lower=-0.25 upper=0.25 effort=0.78125 velocity=0.001
- joint RTseg10_RTseg11_joint: limit lower=-0.25 upper=0.25 effort=1 velocity=0.001 -> lower=-0.25 upper=0.25 effort=0.680555555556 velocity=0.001
- joint RTseg11_RTseg12_joint: limit lower=-0.25 upper=0.25 effort=1 velocity=0.001 -> lower=-0.25 upper=0.25 effort=0.586805555556 velocity=0.001
- joint RTseg1_RTseg2_joint: limit lower=-0.25 upper=0.25 effort=1 velocity=0.001 -> lower=-0.25 upper=0.25 effort=1.83680555556 velocity=0.001
- joint RTseg2_RTseg3_joint: limit lower=-0.25 upper=0.25 effort=1 velocity=0.001 -> lower=-0.25 upper=0.25 effort=1.68055555556 velocity=0.001
- joint RTseg3_RTseg4_joint: limit lower=-0.25 upper=0.25 effort=1 velocity=0.001 -> lower=-0.25 upper=0.25 effort=1.53125 velocity=0.001
- joint RTseg4_RTseg5_joint: limit lower=-0.25 upper=0.25 effort=1 velocity=0.001 -> lower=-0.25 upper=0.25 effort=1.38888888889 velocity=0.001
- joint RTseg5_RTseg6_joint: limit lower=-0.25 upper=0.25 effort=1 velocity=0.001 -> lower=-0.25 upper=0.25 effort=1.25347222222 velocity=0.001
- joint RTseg6_RTseg7_joint: limit lower=-0.25 upper=0.25 effort=1 velocity=0.001 -> lower=-0.25 upper=0.25 effort=1.125 velocity=0.001
- joint RTseg7_RTseg8_joint: limit lower=-0.25 upper=0.25 effort=1 velocity=0.001 -> lower=-0.25 upper=0.25 effort=1.00347222222 velocity=0.001
- joint RTseg8_RTseg9_joint: limit lower=-0.25 upper=0.25 effort=1 velocity=0.001 -> lower=-0.25 upper=0.25 effort=0.888888888889 velocity=0.001
- joint RTseg9_RTseg10_joint: limit lower=-0.25 upper=0.25 effort=1 velocity=0.001 -> lower=-0.25 upper=0.25 effort=0.78125 velocity=0.001
- joint palm_LBseg1_joint: limit lower=-0.1 upper=0.1 effort=1 velocity=0.0001 -> lower=-0.1 upper=0.1 effort=2.0 velocity=0.0001
- joint palm_LTseg1_joint: limit lower=-0.1 upper=0.1 effort=1 velocity=0.0001 -> lower=-0.1 upper=0.1 effort=2.0 velocity=0.0001
- joint palm_RBseg1_joint: limit lower=-0.1 upper=0.1 effort=1 velocity=0.0001 -> lower=-0.1 upper=0.1 effort=2.0 velocity=0.0001
- joint palm_RTseg1_joint: limit lower=-0.1 upper=0.1 effort=1 velocity=0.0001 -> lower=-0.1 upper=0.1 effort=2.0 velocity=0.0001

File: urdf/macros2.xacro (robot description, xacro)
@@ -5,19 +5,19 @@
 <xacro:include filename="$(find main_description)/urdf/inertias.xacro" />
 <xacro:property name="fingerForce" value = "1"/>
-<xacro:macro name="segment" params="name parent length">
-	<xacro:seg name="${name}" length="${length}"/>
-	<xacro:seg_joint seg1="${parent}" seg2="${name}" length="${length}"/>
+<xacro:macro name="segment" params="name parent length height width force">
+	<xacro:seg name="${name}" length="${length}" height="${height}" width="${width}"/>
+	<xacro:seg_joint seg1="${parent}" seg2="${name}" length="${length}" force="${force}"/>
 	<xacro:seg_trans seg1="${parent}" seg2="${name}"/>
 </xacro:macro>
-<xacro:macro name="seg" params="name length">
+<xacro:macro name="seg" params="name length height width">
 	<link name="${name}">
 		<visual>
 			<geometry>
-				<box size="0.02 0.02 ${length}"/>
+				<box size="${width} ${height} ${length}"/>
 			</geometry>
 			<origin xyz="0 0 0"/>
 			<material name="white"/>
 		</visual>
-		<xacro:box_inertial_with_origin x="0.02" y="0.02" z="${length}" mass="0.01">
+		<xacro:box_inertial_with_origin x="${width}" y="${height}" z="${length}" mass="0.01">
 			<origin xyz="0 0 0" rpy="0 0 0"/>
 		</xacro:box_inertial_with_origin>
@@ -30,5 +30,5 @@
 		<collision>
 			<geometry>
-				<box size="0.02 0.02 ${length}"/>
+				<box size="${width} ${height} ${length}"/>
 			</geometry>
 			<origin xyz="0 0 0"/>
@@ -42,8 +42,8 @@
 	</gazebo>
 </xacro:macro>
-<xacro:macro name="seg_joint" params="seg1 seg2 length">
+<xacro:macro name="seg_joint" params="seg1 seg2 length force">
 	<joint name="${seg1}_${seg2}_joint" type="revolute">
 		<axis xyz="1 0 0"/>
-		<limit effort="${fingerForce}" lower="-0.25" upper="0.25" velocity="0.001"/>
+		<limit effort="${force}" lower="-0.25" upper="0.25" velocity="0.001"/>
 		<dynamics damping="0.05" friction="0.0"/>
 		<origin xyz="0 0 ${length}" rpy="0 0 0"/>
@@ -55,8 +55,8 @@
 	</gazebo>
 </xacro:macro>
-<xacro:macro name="seg_joint_offset" params="seg1 seg2 length offset rotation">
+<xacro:macro name="seg_joint_offset" params="seg1 seg2 length offset rotation force">
 	<joint name="${seg1}_${seg2}_joint" type="revolute">
 		<axis xyz="1 0 0"/>
-		<limit effort="${fingerForce}" lower="-0.1" upper="0.1" velocity="0.0001"/>
+		<limit effort="${force}" lower="-0.1" upper="0.1" velocity="0.0001"/>
 		<!--<dynamics damping="0.05" friction="0.0"/>-->
 		<origin xyz="${offset}" rpy="${rotation}"/>

File: urdf/mainDesign.xacro (robot description, xacro)
@@ -38,5 +38,7 @@
 	<base name="palm"/>
 	<length value="0.15"/>
+	<geometry base = "0.02 0.02" tip = "0.01 0.01"/>
 	<origin xyz="0.05 0.05 0" rpy="-0 0 0"/>
+	<force value="2"/>
 </finger>
 <finger name="RT">
@@ -44,5 +46,7 @@
 	<base name="palm"/>
 	<length value="0.15"/>
+	<geometry base = "0.02 0.02" tip = "0.01 0.01"/>
 	<origin xyz="0.05 -0.05 0" rpy="-0 0 3.14159"/>
+	<force value="2"/>
 </finger>
 <finger name="LB">
@@ -50,11 +54,15 @@
 	<base name="palm"/>
 	<length value="0.15"/>
+	<geometry base = "0.02 0.02" tip = "0.01 0.01"/>
 	<origin xyz="-0.05 0.05 0" rpy="-0 0 0"/>
+	<force value="2"/>
 </finger>
 <finger name="RB">
 	<segments value="12"/>
 	<base name="palm"/>
+	<geometry base = "0.02 0.02" tip = "0.01 0.01"/>
 	<length value="0.15"/>
 	<origin xyz="-0.05 -0.05 0" rpy="-0 0 3.14159"/>
+	<force value="2"/>
 </finger>
 <gazebo>
