Commit message: Gripper position estimation
rough estimation from stess/strain sensors

File: urdf/output.xacro (robot description, xacro)
@@ -37,62 +37,62 @@
 </gazebo>
  <!--  MACROS FOR FINGER: LT-->
-<xacro:seg name="LTseg1" length="0.0125"/>
-<xacro:seg_joint_offset seg1="palm" seg2="LTseg1" length="0.0125" offset="0.05 0.05 0" rotation="-0 0 0" />
+<xacro:seg name= "LTseg1" length = "0.0125" height = "0.02" width = "0.02" />
+<xacro:seg_joint_offset seg1= "palm" seg2="LTseg1" length="0.0125" offset="0.05 0.05 0" rotation="-0 0 0" force="2.0" />
 <xacro:seg_trans seg1="palm" seg2="LTseg1"/>
-<xacro:segment name="LTseg2" parent="LTseg1" length="0.0125"/>
-<xacro:segment name="LTseg3" parent="LTseg2" length="0.0125"/>
-<xacro:segment name="LTseg4" parent="LTseg3" length="0.0125"/>
-<xacro:segment name="LTseg5" parent="LTseg4" length="0.0125"/>
-<xacro:segment name="LTseg6" parent="LTseg5" length="0.0125"/>
-<xacro:segment name="LTseg7" parent="LTseg6" length="0.0125"/>
-<xacro:segment name="LTseg8" parent="LTseg7" length="0.0125"/>
-<xacro:segment name="LTseg9" parent="LTseg8" length="0.0125"/>
-<xacro:segment name="LTseg10" parent="LTseg9" length="0.0125"/>
-<xacro:segment name="LTseg11" parent="LTseg10" length="0.0125"/>
-<xacro:segment name="LTseg12" parent="LTseg11" length="0.0125"/>
+<xacro:segment name= "LTseg2" parent="LTseg1" length="0.0125" height="0.0191666666667" width = "0.0191666666667" force = "1.83680555556" />
+<xacro:segment name= "LTseg3" parent="LTseg2" length="0.0125" height="0.0183333333333" width = "0.0183333333333" force = "1.68055555556" />
+<xacro:segment name= "LTseg4" parent="LTseg3" length="0.0125" height="0.0175" width = "0.0175" force = "1.53125" />
+<xacro:segment name= "LTseg5" parent="LTseg4" length="0.0125" height="0.0166666666667" width = "0.0166666666667" force = "1.38888888889" />
+<xacro:segment name= "LTseg6" parent="LTseg5" length="0.0125" height="0.0158333333333" width = "0.0158333333333" force = "1.25347222222" />
+<xacro:segment name= "LTseg7" parent="LTseg6" length="0.0125" height="0.015" width = "0.015" force = "1.125" />
+<xacro:segment name= "LTseg8" parent="LTseg7" length="0.0125" height="0.0141666666667" width = "0.0141666666667" force = "1.00347222222" />
+<xacro:segment name= "LTseg9" parent="LTseg8" length="0.0125" height="0.0133333333333" width = "0.0133333333333" force = "0.888888888889" />
+<xacro:segment name= "LTseg10" parent="LTseg9" length="0.0125" height="0.0125" width = "0.0125" force = "0.78125" />
+<xacro:segment name= "LTseg11" parent="LTseg10" length="0.0125" height="0.0116666666667" width = "0.0116666666667" force = "0.680555555556" />
+<xacro:segment name= "LTseg12" parent="LTseg11" length="0.0125" height="0.0108333333333" width = "0.0108333333333" force = "0.586805555556" />
  <!--  MACROS FOR FINGER: RT-->
-<xacro:seg name="RTseg1" length="0.0125"/>
-<xacro:seg_joint_offset seg1="palm" seg2="RTseg1" length="0.0125" offset="0.05 -0.05 0" rotation="-0 0 3.14159" />
+<xacro:seg name= "RTseg1" length = "0.0125" height = "0.02" width = "0.02" />
+<xacro:seg_joint_offset seg1= "palm" seg2="RTseg1" length="0.0125" offset="0.05 -0.05 0" rotation="-0 0 3.14159" force="2.0" />
 <xacro:seg_trans seg1="palm" seg2="RTseg1"/>
-<xacro:segment name="RTseg2" parent="RTseg1" length="0.0125"/>
-<xacro:segment name="RTseg3" parent="RTseg2" length="0.0125"/>
-<xacro:segment name="RTseg4" parent="RTseg3" length="0.0125"/>
-<xacro:segment name="RTseg5" parent="RTseg4" length="0.0125"/>
-<xacro:segment name="RTseg6" parent="RTseg5" length="0.0125"/>
-<xacro:segment name="RTseg7" parent="RTseg6" length="0.0125"/>
-<xacro:segment name="RTseg8" parent="RTseg7" length="0.0125"/>
-<xacro:segment name="RTseg9" parent="RTseg8" length="0.0125"/>
-<xacro:segment name="RTseg10" parent="RTseg9" length="0.0125"/>
-<xacro:segment name="RTseg11" parent="RTseg10" length="0.0125"/>
-<xacro:segment name="RTseg12" parent="RTseg11" length="0.0125"/>
+<xacro:segment name= "RTseg2" parent="RTseg1" length="0.0125" height="0.0191666666667" width = "0.0191666666667" force = "1.83680555556" />
+<xacro:segment name= "RTseg3" parent="RTseg2" length="0.0125" height="0.0183333333333" width = "0.0183333333333" force = "1.68055555556" />
+<xacro:segment name= "RTseg4" parent="RTseg3" length="0.0125" height="0.0175" width = "0.0175" force = "1.53125" />
+<xacro:segment name= "RTseg5" parent="RTseg4" length="0.0125" height="0.0166666666667" width = "0.0166666666667" force = "1.38888888889" />
+<xacro:segment name= "RTseg6" parent="RTseg5" length="0.0125" height="0.0158333333333" width = "0.0158333333333" force = "1.25347222222" />
+<xacro:segment name= "RTseg7" parent="RTseg6" length="0.0125" height="0.015" width = "0.015" force = "1.125" />
+<xacro:segment name= "RTseg8" parent="RTseg7" length="0.0125" height="0.0141666666667" width = "0.0141666666667" force = "1.00347222222" />
+<xacro:segment name= "RTseg9" parent="RTseg8" length="0.0125" height="0.0133333333333" width = "0.0133333333333" force = "0.888888888889" />
+<xacro:segment name= "RTseg10" parent="RTseg9" length="0.0125" height="0.0125" width = "0.0125" force = "0.78125" />
+<xacro:segment name= "RTseg11" parent="RTseg10" length="0.0125" height="0.0116666666667" width = "0.0116666666667" force = "0.680555555556" />
+<xacro:segment name= "RTseg12" parent="RTseg11" length="0.0125" height="0.0108333333333" width = "0.0108333333333" force = "0.586805555556" />
  <!--  MACROS FOR FINGER: LB-->
-<xacro:seg name="LBseg1" length="0.0125"/>
-<xacro:seg_joint_offset seg1="palm" seg2="LBseg1" length="0.0125" offset="-0.05 0.05 0" rotation="-0 0 0" />
+<xacro:seg name= "LBseg1" length = "0.0125" height = "0.02" width = "0.02" />
+<xacro:seg_joint_offset seg1= "palm" seg2="LBseg1" length="0.0125" offset="-0.05 0.05 0" rotation="-0 0 0" force="2.0" />
 <xacro:seg_trans seg1="palm" seg2="LBseg1"/>
-<xacro:segment name="LBseg2" parent="LBseg1" length="0.0125"/>
-<xacro:segment name="LBseg3" parent="LBseg2" length="0.0125"/>
-<xacro:segment name="LBseg4" parent="LBseg3" length="0.0125"/>
-<xacro:segment name="LBseg5" parent="LBseg4" length="0.0125"/>
-<xacro:segment name="LBseg6" parent="LBseg5" length="0.0125"/>
-<xacro:segment name="LBseg7" parent="LBseg6" length="0.0125"/>
-<xacro:segment name="LBseg8" parent="LBseg7" length="0.0125"/>
-<xacro:segment name="LBseg9" parent="LBseg8" length="0.0125"/>
-<xacro:segment name="LBseg10" parent="LBseg9" length="0.0125"/>
-<xacro:segment name="LBseg11" parent="LBseg10" length="0.0125"/>
-<xacro:segment name="LBseg12" parent="LBseg11" length="0.0125"/>
+<xacro:segment name= "LBseg2" parent="LBseg1" length="0.0125" height="0.0191666666667" width = "0.0191666666667" force = "1.83680555556" />
+<xacro:segment name= "LBseg3" parent="LBseg2" length="0.0125" height="0.0183333333333" width = "0.0183333333333" force = "1.68055555556" />
+<xacro:segment name= "LBseg4" parent="LBseg3" length="0.0125" height="0.0175" width = "0.0175" force = "1.53125" />
+<xacro:segment name= "LBseg5" parent="LBseg4" length="0.0125" height="0.0166666666667" width = "0.0166666666667" force = "1.38888888889" />
+<xacro:segment name= "LBseg6" parent="LBseg5" length="0.0125" height="0.0158333333333" width = "0.0158333333333" force = "1.25347222222" />
+<xacro:segment name= "LBseg7" parent="LBseg6" length="0.0125" height="0.015" width = "0.015" force = "1.125" />
+<xacro:segment name= "LBseg8" parent="LBseg7" length="0.0125" height="0.0141666666667" width = "0.0141666666667" force = "1.00347222222" />
+<xacro:segment name= "LBseg9" parent="LBseg8" length="0.0125" height="0.0133333333333" width = "0.0133333333333" force = "0.888888888889" />
+<xacro:segment name= "LBseg10" parent="LBseg9" length="0.0125" height="0.0125" width = "0.0125" force = "0.78125" />
+<xacro:segment name= "LBseg11" parent="LBseg10" length="0.0125" height="0.0116666666667" width = "0.0116666666667" force = "0.680555555556" />
+<xacro:segment name= "LBseg12" parent="LBseg11" length="0.0125" height="0.0108333333333" width = "0.0108333333333" force = "0.586805555556" />
  <!--  MACROS FOR FINGER: RB-->
-<xacro:seg name="RBseg1" length="0.0125"/>
-<xacro:seg_joint_offset seg1="palm" seg2="RBseg1" length="0.0125" offset="-0.05 -0.05 0" rotation="-0 0 3.14159" />
+<xacro:seg name= "RBseg1" length = "0.0125" height = "0.02" width = "0.02" />
+<xacro:seg_joint_offset seg1= "palm" seg2="RBseg1" length="0.0125" offset="-0.05 -0.05 0" rotation="-0 0 3.14159" force="2.0" />
 <xacro:seg_trans seg1="palm" seg2="RBseg1"/>
-<xacro:segment name="RBseg2" parent="RBseg1" length="0.0125"/>
-<xacro:segment name="RBseg3" parent="RBseg2" length="0.0125"/>
-<xacro:segment name="RBseg4" parent="RBseg3" length="0.0125"/>
-<xacro:segment name="RBseg5" parent="RBseg4" length="0.0125"/>
-<xacro:segment name="RBseg6" parent="RBseg5" length="0.0125"/>
-<xacro:segment name="RBseg7" parent="RBseg6" length="0.0125"/>
-<xacro:segment name="RBseg8" parent="RBseg7" length="0.0125"/>
-<xacro:segment name="RBseg9" parent="RBseg8" length="0.0125"/>
-<xacro:segment name="RBseg10" parent="RBseg9" length="0.0125"/>
-<xacro:segment name="RBseg11" parent="RBseg10" length="0.0125"/>
-<xacro:segment name="RBseg12" parent="RBseg11" length="0.0125"/>
+<xacro:segment name= "RBseg2" parent="RBseg1" length="0.0125" height="0.0191666666667" width = "0.0191666666667" force = "1.83680555556" />
+<xacro:segment name= "RBseg3" parent="RBseg2" length="0.0125" height="0.0183333333333" width = "0.0183333333333" force = "1.68055555556" />
+<xacro:segment name= "RBseg4" parent="RBseg3" length="0.0125" height="0.0175" width = "0.0175" force = "1.53125" />
+<xacro:segment name= "RBseg5" parent="RBseg4" length="0.0125" height="0.0166666666667" width = "0.0166666666667" force = "1.38888888889" />
+<xacro:segment name= "RBseg6" parent="RBseg5" length="0.0125" height="0.0158333333333" width = "0.0158333333333" force = "1.25347222222" />
+<xacro:segment name= "RBseg7" parent="RBseg6" length="0.0125" height="0.015" width = "0.015" force = "1.125" />
+<xacro:segment name= "RBseg8" parent="RBseg7" length="0.0125" height="0.0141666666667" width = "0.0141666666667" force = "1.00347222222" />
+<xacro:segment name= "RBseg9" parent="RBseg8" length="0.0125" height="0.0133333333333" width = "0.0133333333333" force = "0.888888888889" />
+<xacro:segment name= "RBseg10" parent="RBseg9" length="0.0125" height="0.0125" width = "0.0125" force = "0.78125" />
+<xacro:segment name= "RBseg11" parent="RBseg10" length="0.0125" height="0.0116666666667" width = "0.0116666666667" force = "0.680555555556" />
+<xacro:segment name= "RBseg12" parent="RBseg11" length="0.0125" height="0.0108333333333" width = "0.0108333333333" force = "0.586805555556" />
 </robot>
