Commit message: Test worlds, position error log, multiple gripper control types

File: urdf/macros2.xacro (robot description, xacro)
@@ -28,5 +28,5 @@
 		</inertial>
 		-->
-		<collision>
+		<collision name="${name}_collision">
 			<geometry>
 				<box size="${width} ${height} ${length}"/>
@@ -41,4 +41,11 @@
 		<selfCollide>true</selfCollide>
 		<gravity>true</gravity>
+		<sensor name = "${name}_sensor" type="contact">
+			<always_on>true</always_on>
+			<contact>
+				<collision>${name}_collision</collision>
+			</contact>
+			<update_rate> 30 </update_rate>
+		</sensor>
 	</gazebo>
 </xacro:macro>
