Commit message: new URDF added

File: scripts/output.xacro (robot description, xacro)
@@ -26,8 +26,8 @@
 	<gravity>true</gravity>
 </gazebo>
-<joint name="palm_world_joint" type="fixed">
-    <parent link="arm3_1" />
+<joint name="palm_arm_joint" type="fixed">
+    <parent link="Link4_1" />
     <child link="palm" />
-	<origin rpy="0 ${3.14/2} 0" xyz="0.1 0 0" />
+	<origin rpy="0 0 0" xyz="0.0 0 0.12" />
 </joint>
 <gazebo>

File: urdf/arm.xacro (robot description, xacro)
@@ -9,5 +9,150 @@
 <xacro:property name="damping" value = "0"/>
 <xacro:property name="offset" value="-0.05"/>
-<!--  LINKS  -->
+<!-- LINKS  -->
+<!--<xacro:include filename="$(find design2_description)/urdf/materials.xacro" />-->
+<!--<xacro:include filename="$(find design2_description)/urdf/design2.trans" />-->
+<!--<xacro:include filename="$(find design2_description)/urdf/design2.gazebo" />-->
+<link name="base_link">
+  <inertial>
+    <origin rpy="0 0 0" xyz="-3.054172551678278e-15 2.5451437930652316e-17 0.009826233848161996"/>
+    <mass value="2.1038693653686527"/>
+    <inertia ixx="0.002498" ixy="0.0" ixz="-0.0" iyy="0.002498" iyz="0.0" izz="0.004751"/>
+  </inertial>
+  <visual>
+    <origin rpy="0 0 0" xyz="0 0 0"/>
+    <geometry>
+      <mesh filename="package://main_description/meshes/base_link.stl" scale="0.001 0.001 0.001"/>
+    </geometry>
+    <material name="silver"/>
+  </visual>
+  <collision>
+    <origin rpy="0 0 0" xyz="0 0 0"/>
+    <geometry>
+      <mesh filename="package://main_description/meshes/base_link.stl" scale="0.001 0.001 0.001"/>
+    </geometry>
+  </collision>
+</link>
+<link name="Link1_1">
+  <inertial>
+    <origin rpy="0 0 0" xyz="-6.1328821587432384e-06 0.007231132282278709 0.010400791755463774"/>
+    <mass value="0.8688143187550561"/>
+    <inertia ixx="0.000613" ixy="0.0" ixz="0.0" iyy="0.000486" iyz="-8.3e-05" izz="0.000932"/>
+  </inertial>
+  <visual>
+    <origin rpy="0 0 0" xyz="-0.0 -0.0 -0.025"/>
+    <geometry>
+      <mesh filename="package://main_description/meshes/Link1_1.stl" scale="0.001 0.001 0.001"/>
+    </geometry>
+    <material name="silver"/>
+  </visual>
+  <collision>
+    <origin rpy="0 0 0" xyz="-0.0 -0.0 -0.025"/>
+    <geometry>
+      <mesh filename="package://main_description/meshes/Link1_1.stl" scale="0.001 0.001 0.001"/>
+    </geometry>
+  </collision>
+</link>
+<link name="Link2_1">
+  <inertial>
+    <origin rpy="0 0 0" xyz="-1.4589717024326475e-07 0.009220625083884316 0.09374198522195988"/>
+    <mass value="0.6628237762897414"/>
+    <inertia ixx="0.002038" ixy="0.0" ixz="0.0" iyy="0.001955" iyz="-0.000356" izz="0.000168"/>
+  </inertial>
+  <visual>
+    <origin rpy="0 0 0" xyz="2.1e-05 -0.004903 -0.05"/>
+    <geometry>
+      <mesh filename="package://main_description/meshes/Link2_1.stl" scale="0.001 0.001 0.001"/>
+    </geometry>
+    <material name="silver"/>
+  </visual>
+  <collision>
+    <origin rpy="0 0 0" xyz="2.1e-05 -0.004903 -0.05"/>
+    <geometry>
+      <mesh filename="package://main_description/meshes/Link2_1.stl" scale="0.001 0.001 0.001"/>
+    </geometry>
+  </collision>
+</link>
+<link name="Link3_1">
+  <inertial>
+    <origin rpy="0 0 0" xyz="1.9618427109714154e-05 0.006527757535011174 0.07498286609368165"/>
+    <mass value="0.4910812167638009"/>
+    <inertia ixx="0.001039" ixy="-0.0" ixz="-0.0" iyy="0.001007" iyz="-0.000178" izz="8.5e-05"/>
+  </inertial>
+  <visual>
+    <origin rpy="0 0 0" xyz="2.1e-05 -0.004903 -0.2"/>
+    <geometry>
+      <mesh filename="package://main_description/meshes/Link3_1.stl" scale="0.001 0.001 0.001"/>
+    </geometry>
+    <material name="silver"/>
+  </visual>
+  <collision>
+    <origin rpy="0 0 0" xyz="2.1e-05 -0.004903 -0.2"/>
+    <geometry>
+      <mesh filename="package://main_description/meshes/Link3_1.stl" scale="0.001 0.001 0.001"/>
+    </geometry>
+  </collision>
+</link>
+<link name="Link4_1">
+  <inertial>
+    <origin rpy="0 0 0" xyz="-1.842082955655732e-07 -0.004999749873264598 0.032486936025046875"/>
+    <mass value="0.16819090005804693"/>
+    <inertia ixx="0.000103" ixy="0.0" ixz="0.0" iyy="0.00011" iyz="0.0" izz="1e-05"/>
+  </inertial>
+  <visual>
+    <origin rpy="0 0 0" xyz="-1.2e-05 -0.004903 -0.325"/>
+    <geometry>
+      <mesh filename="package://main_description/meshes/Link4_1.stl" scale="0.001 0.001 0.001"/>
+    </geometry>
+    <material name="silver"/>
+  </visual>
+  <collision>
+    <origin rpy="0 0 0" xyz="-1.2e-05 -0.004903 -0.325"/>
+    <geometry>
+      <mesh filename="package://main_description/meshes/Link4_1.stl" scale="0.001 0.001 0.001"/>
+    </geometry>
+  </collision>
+</link>
+<!--  JOINTS  -->
+<joint name="world_joint" type="fixed">
+  <axis xyz="0 0 1"/>
+	<origin xyz="0.0 0.0 0.0" rpy="0 0 0" />
+	<parent link="world"/>
+	<child link="base_link"/>
+</joint>
+<joint name="Rev1" type="continuous">
+  <origin rpy="0 0 0" xyz="0.0 0.0 0.025"/>
+  <parent link="base_link"/>
+  <child link="Link1_1"/>
+  <axis xyz="0.0 0.0 1.0"/>
+  <limit effort="${strength}" lower="0.0" upper="6.283185" velocity="${speed}"/>
+  <dynamics damping="${damping}" friction="0.0"/>
+</joint>
+<joint name="Rev2" type="revolute">
+  <origin rpy="0 0 0" xyz="-2.1e-05 0.004903 0.025"/>
+  <parent link="Link1_1"/>
+  <child link="Link2_1"/>
+  <axis xyz="0.0 -1.0 0.0"/>
+  <limit effort="${strength}" lower="-1.396263" upper="1.396263" velocity="${speed}"/>
+  <dynamics damping="${damping}" friction="0.0"/>
+</joint>
+<joint name="Rev3" type="revolute">
+  <origin rpy="0 0 0" xyz="0.0 0.0 0.15"/>
+  <parent link="Link2_1"/>
+  <child link="Link3_1"/>
+  <axis xyz="0.0 -1.0 0.0"/>
+  <limit effort="${strength}" lower="-2.792527" upper="2.792527" velocity="${speed}"/>
+  <dynamics damping="${damping}" friction="0.0"/>
+</joint>
+<joint name="Rev4" type="revolute">
+  <origin rpy="0 0 0" xyz="3.3e-05 0.0 0.125"/>
+  <parent link="Link3_1"/>
+  <child link="Link4_1"/>
+  <axis xyz="0.0 -1.0 0.0"/>
+  <limit effort="${strength}" lower="-2.617994" upper="2.617994" velocity="${speed}"/>
+  <dynamics damping="${damping}" friction="0.0"/>
+</joint>
+</robot>
+<!--
+  LINKS
 <joint name="anchor" type="continuous">
   <axis xyz="0 0 1"/>
@@ -98,5 +243,4 @@
   </collision>
 </link>
-<!--
 <link name="HandBase_1">
   <inertial>
@@ -138,6 +282,5 @@
     </geometry>
   </collision>
-</link> -->
-<!--- JOINTS  -->
+</link>
 <joint name="base_link" type="revolute">
   <origin rpy="0 0 0" xyz="0.0 0.0 0.036536"/>
@@ -164,5 +307,4 @@
   <dynamics damping="${damping}" friction="0.0"/>
 </joint>
-<!--
 <joint name="Joint4" type="revolute">
   <origin rpy="0 0 0" xyz="0.065 -0.015 0.0"/>
@@ -178,4 +320,5 @@
   <axis xyz="0.0 1.0 0.0"/>
   <limit effort="${strength}" lower="-0.085" upper="0.0" velocity="100"/>
-</joint> -->
+</joint>
 </robot>
+-->

File: urdf/description_log.urdf (robot description, URDF)
Before this commit: robot Design, 54 links, 53 joints
Links:
- removed link arm1_1
- removed link arm2_1
- removed link arm3_1
- added link Link1_1, mass 0.8688143187550561; collision mesh filename=package://main_description/meshes/Link1_1.stl scale=0.001 0.001 0.001; visual mesh filename=package://main_description/meshes/Link1_1.stl scale=0.001 0.001 0.001
- added link Link2_1, mass 0.6628237762897414; collision mesh filename=package://main_description/meshes/Link2_1.stl scale=0.001 0.001 0.001; visual mesh filename=package://main_description/meshes/Link2_1.stl scale=0.001 0.001 0.001
- added link Link3_1, mass 0.4910812167638009; collision mesh filename=package://main_description/meshes/Link3_1.stl scale=0.001 0.001 0.001; visual mesh filename=package://main_description/meshes/Link3_1.stl scale=0.001 0.001 0.001
- added link Link4_1, mass 0.16819090005804693; collision mesh filename=package://main_description/meshes/Link4_1.stl scale=0.001 0.001 0.001; visual mesh filename=package://main_description/meshes/Link4_1.stl scale=0.001 0.001 0.001
- link base_link: mass 1.526896640260832 -> 2.1038693653686527; geometry collision mesh filename=package://main_description/meshes/base_link.stl scale=0.001 0.001 0.001; visual mesh filename=package://main_description/meshes/base_link.stl scale=0.001 0.001 0.001
Joints:
- removed joint Joint2
- removed joint Joint3
- removed joint anchor
- removed joint base_link
- removed joint palm_world_joint
- added joint Rev1: type continuous, parent base_link, child Link1_1, origin xyz=0.0 0.0 0.025 rpy=0 0 0, axis 0.0 0.0 1.0, limit lower=0.0 upper=6.283185 effort=1000 velocity=0.01
- added joint Rev2: type revolute, parent Link1_1, child Link2_1, origin xyz=-2.1e-05 0.004903 0.025 rpy=0 0 0, axis 0.0 -1.0 0.0, limit lower=-1.396263 upper=1.396263 effort=1000 velocity=0.01
- added joint Rev3: type revolute, parent Link2_1, child Link3_1, origin xyz=0.0 0.0 0.15 rpy=0 0 0, axis 0.0 -1.0 0.0, limit lower=-2.792527 upper=2.792527 effort=1000 velocity=0.01
- added joint Rev4: type revolute, parent Link3_1, child Link4_1, origin xyz=3.3e-05 0.0 0.125 rpy=0 0 0, axis 0.0 -1.0 0.0, limit lower=-2.617994 upper=2.617994 effort=1000 velocity=0.01
- added joint palm_arm_joint: type fixed, parent Link4_1, child palm, origin xyz=0.0 0 0.12 rpy=0 0 0
- added joint world_joint: type fixed, parent world, child base_link, origin xyz=0.0 0.0 0.0 rpy=0 0 0, axis 0 0 1

File: urdf/mainDesign.xacro (robot description, xacro)
@@ -29,8 +29,8 @@
 	<gravity>true</gravity>
 </gazebo>
-<joint name="palm_world_joint" type="fixed">
-    <parent link="arm3_1"/>
+<joint name="palm_arm_joint" type="fixed">
+    <parent link="Link4_1"/>
     <child link="palm"/>
-	<origin xyz="0.1 0 0" rpy="0 ${3.14/2} 0"/>
+	<origin xyz="0.0 0 0.12" rpy="0 0 0"/>
 </joint>
 <finger name="LT">

File: urdf/output.xacro (robot description, xacro)
@@ -26,8 +26,8 @@
 	<gravity>true</gravity>
 </gazebo>
-<joint name="palm_world_joint" type="fixed">
-    <parent link="arm3_1" />
+<joint name="palm_arm_joint" type="fixed">
+    <parent link="Link4_1" />
     <child link="palm" />
-	<origin rpy="0 ${3.14/2} 0" xyz="0.1 0 0" />
+	<origin rpy="0 0 0" xyz="0.0 0 0.12" />
 </joint>
 <gazebo>

Commit message: Expanded path planning and larger model

File: scripts/output.xacro (robot description, xacro)
@@ -29,5 +29,5 @@
     <parent link="Link4_1" />
     <child link="palm" />
-	<origin rpy="0 0 0" xyz="0.0 0 0.12" />
+	<origin rpy="0 0 0" xyz="0.0 0 0.15" />
 </joint>
 <gazebo>

File: urdf/arm.xacro (robot description, xacro)
@@ -15,7 +15,7 @@
 <link name="base_link">
   <inertial>
-    <origin rpy="0 0 0" xyz="-3.054172551678278e-15 2.5451437930652316e-17 0.009826233848161996"/>
-    <mass value="2.1038693653686527"/>
-    <inertia ixx="0.002498" ixy="0.0" ixz="-0.0" iyy="0.002498" iyz="0.0" izz="0.004751"/>
+    <origin rpy="0 0 0" xyz="-6.108345103356556e-15 5.090287586130463e-17 0.01965246769632399"/>
+    <mass value="16.83095492294922"/>
+    <inertia ixx="0.079936" ixy="0.0" ixz="-0.0" iyy="0.079936" iyz="0.0" izz="0.152021"/>
   </inertial>
   <visual>
@@ -35,10 +35,10 @@
 <link name="Link1_1">
   <inertial>
-    <origin rpy="0 0 0" xyz="-6.1328821587432384e-06 0.007231132282278709 0.010400791755463774"/>
-    <mass value="0.8688143187550561"/>
-    <inertia ixx="0.000613" ixy="0.0" ixz="0.0" iyy="0.000486" iyz="-8.3e-05" izz="0.000932"/>
-  </inertial>
-  <visual>
-    <origin rpy="0 0 0" xyz="-0.0 -0.0 -0.025"/>
+    <origin rpy="0 0 0" xyz="-1.2279118486616705e-05 0.01442476351451121 0.020602870891923072"/>
+    <mass value="0.9178712114753625"/>
+    <inertia ixx="0.002553" ixy="0.0" ixz="0.0" iyy="0.002018" iyz="-0.00035" izz="0.00387"/>
+  </inertial>
+  <visual>
+    <origin rpy="0 0 0" xyz="-0.0 -0.0 -0.05"/>
     <geometry>
       <mesh filename="package://main_description/meshes/Link1_1.stl" scale="0.001 0.001 0.001"/>
@@ -47,5 +47,5 @@
   </visual>
   <collision>
-    <origin rpy="0 0 0" xyz="-0.0 -0.0 -0.025"/>
+    <origin rpy="0 0 0" xyz="-0.0 -0.0 -0.05"/>
     <geometry>
       <mesh filename="package://main_description/meshes/Link1_1.stl" scale="0.001 0.001 0.001"/>
@@ -55,10 +55,10 @@
 <link name="Link2_1">
   <inertial>
-    <origin rpy="0 0 0" xyz="-1.4589717024326475e-07 0.009220625083884316 0.09374198522195988"/>
-    <mass value="0.6628237762897414"/>
-    <inertia ixx="0.002038" ixy="0.0" ixz="0.0" iyy="0.001955" iyz="-0.000356" izz="0.000168"/>
-  </inertial>
-  <visual>
-    <origin rpy="0 0 0" xyz="2.1e-05 -0.004903 -0.05"/>
+    <origin rpy="0 0 0" xyz="-2.968335648842978e-07 0.018054267252499347 0.1868568711048091"/>
+    <mass value="0.712050673323837"/>
+    <inertia ixx="0.008737" ixy="0.0" ixz="0.0" iyy="0.008392" iyz="-0.001509" izz="0.000705"/>
+  </inertial>
+  <visual>
+    <origin rpy="0 0 0" xyz="4.2e-05 -0.009807 -0.1"/>
     <geometry>
       <mesh filename="package://main_description/meshes/Link2_1.stl" scale="0.001 0.001 0.001"/>
@@ -67,5 +67,5 @@
   </visual>
   <collision>
-    <origin rpy="0 0 0" xyz="2.1e-05 -0.004903 -0.05"/>
+    <origin rpy="0 0 0" xyz="4.2e-05 -0.009807 -0.1"/>
     <geometry>
       <mesh filename="package://main_description/meshes/Link2_1.stl" scale="0.001 0.001 0.001"/>
@@ -75,10 +75,10 @@
 <link name="Link3_1">
   <inertial>
-    <origin rpy="0 0 0" xyz="1.9618427109714154e-05 0.006527757535011174 0.07498286609368165"/>
-    <mass value="0.4910812167638009"/>
-    <inertia ixx="0.001039" ixy="-0.0" ixz="-0.0" iyy="0.001007" iyz="-0.000178" izz="8.5e-05"/>
-  </inertial>
-  <visual>
-    <origin rpy="0 0 0" xyz="2.1e-05 -0.004903 -0.2"/>
+    <origin rpy="0 0 0" xyz="3.894856228585856e-05 0.012744269230917583 0.14887041213898544"/>
+    <mass value="0.5352959751924613"/>
+    <inertia ixx="0.004471" ixy="-0.0" ixz="-1e-06" iyy="0.004348" iyz="-0.000747" izz="0.000361"/>
+  </inertial>
+  <visual>
+    <origin rpy="0 0 0" xyz="4.2e-05 -0.009807 -0.4"/>
     <geometry>
       <mesh filename="package://main_description/meshes/Link3_1.stl" scale="0.001 0.001 0.001"/>
@@ -87,5 +87,5 @@
   </visual>
   <collision>
-    <origin rpy="0 0 0" xyz="2.1e-05 -0.004903 -0.2"/>
+    <origin rpy="0 0 0" xyz="4.2e-05 -0.009807 -0.4"/>
     <geometry>
       <mesh filename="package://main_description/meshes/Link3_1.stl" scale="0.001 0.001 0.001"/>
@@ -95,10 +95,10 @@
 <link name="Link4_1">
   <inertial>
-    <origin rpy="0 0 0" xyz="-1.842082955655732e-07 -0.004999749873264598 0.032486936025046875"/>
-    <mass value="0.16819090005804693"/>
-    <inertia ixx="0.000103" ixy="0.0" ixz="0.0" iyy="0.00011" iyz="0.0" izz="1e-05"/>
-  </inertial>
-  <visual>
-    <origin rpy="0 0 0" xyz="-1.2e-05 -0.004903 -0.325"/>
+    <origin rpy="0 0 0" xyz="-3.684166078735014e-07 -0.010000499675700233 0.06497387205009375"/>
+    <mass value="0.18168902324741887"/>
+    <inertia ixx="0.000446" ixy="0.0" ixz="0.0" iyy="0.000477" iyz="0.0" izz="4.3e-05"/>
+  </inertial>
+  <visual>
+    <origin rpy="0 0 0" xyz="-2.4e-05 -0.009807 -0.65"/>
     <geometry>
       <mesh filename="package://main_description/meshes/Link4_1.stl" scale="0.001 0.001 0.001"/>
@@ -107,5 +107,5 @@
   </visual>
   <collision>
-    <origin rpy="0 0 0" xyz="-1.2e-05 -0.004903 -0.325"/>
+    <origin rpy="0 0 0" xyz="-2.4e-05 -0.009807 -0.65"/>
     <geometry>
       <mesh filename="package://main_description/meshes/Link4_1.stl" scale="0.001 0.001 0.001"/>
@@ -121,5 +121,5 @@
 </joint>
 <joint name="Rev1" type="continuous">
-  <origin rpy="0 0 0" xyz="0.0 0.0 0.025"/>
+  <origin rpy="0 0 0" xyz="0.0 0.0 0.05"/>
   <parent link="base_link"/>
   <child link="Link1_1"/>
@@ -129,5 +129,5 @@
 </joint>
 <joint name="Rev2" type="revolute">
-  <origin rpy="0 0 0" xyz="-2.1e-05 0.004903 0.025"/>
+  <origin rpy="0 0 0" xyz="-4.2e-05 0.009807 0.05"/>
   <parent link="Link1_1"/>
   <child link="Link2_1"/>
@@ -137,5 +137,5 @@
 </joint>
 <joint name="Rev3" type="revolute">
-  <origin rpy="0 0 0" xyz="0.0 0.0 0.15"/>
+  <origin rpy="0 0 0" xyz="0.0 0.0 0.3"/>
   <parent link="Link2_1"/>
   <child link="Link3_1"/>
@@ -145,5 +145,5 @@
 </joint>
 <joint name="Rev4" type="revolute">
-  <origin rpy="0 0 0" xyz="3.3e-05 0.0 0.125"/>
+  <origin rpy="0 0 0" xyz="6.6e-05 0.0 0.25"/>
   <parent link="Link3_1"/>
   <child link="Link4_1"/>

File: urdf/description_log.urdf (robot description, URDF)
Before this commit: robot Design, 55 links, 54 joints
Links:
- link Link1_1: mass 0.8688143187550561 -> 0.9178712114753625
- link Link2_1: mass 0.6628237762897414 -> 0.712050673323837
- link Link3_1: mass 0.4910812167638009 -> 0.5352959751924613
- link Link4_1: mass 0.16819090005804693 -> 0.18168902324741887
- link base_link: mass 2.1038693653686527 -> 16.83095492294922
Joints:
- joint LBseg10_LBseg11_joint: origin xyz=0 0 0.0175 rpy=0 0 0 -> xyz=0 0 0.0125 rpy=0 0 0
- joint LBseg11_LBseg12_joint: origin xyz=0 0 0.0175 rpy=0 0 0 -> xyz=0 0 0.0125 rpy=0 0 0
- joint LBseg1_LBseg2_joint: origin xyz=0 0 0.0175 rpy=0 0 0 -> xyz=0 0 0.0125 rpy=0 0 0
- joint LBseg2_LBseg3_joint: origin xyz=0 0 0.0175 rpy=0 0 0 -> xyz=0 0 0.0125 rpy=0 0 0
- joint LBseg3_LBseg4_joint: origin xyz=0 0 0.0175 rpy=0 0 0 -> xyz=0 0 0.0125 rpy=0 0 0
- joint LBseg4_LBseg5_joint: origin xyz=0 0 0.0175 rpy=0 0 0 -> xyz=0 0 0.0125 rpy=0 0 0
- joint LBseg5_LBseg6_joint: origin xyz=0 0 0.0175 rpy=0 0 0 -> xyz=0 0 0.0125 rpy=0 0 0
- joint LBseg6_LBseg7_joint: origin xyz=0 0 0.0175 rpy=0 0 0 -> xyz=0 0 0.0125 rpy=0 0 0
- joint LBseg7_LBseg8_joint: origin xyz=0 0 0.0175 rpy=0 0 0 -> xyz=0 0 0.0125 rpy=0 0 0
- joint LBseg8_LBseg9_joint: origin xyz=0 0 0.0175 rpy=0 0 0 -> xyz=0 0 0.0125 rpy=0 0 0
- joint LBseg9_LBseg10_joint: origin xyz=0 0 0.0175 rpy=0 0 0 -> xyz=0 0 0.0125 rpy=0 0 0
- joint LTseg10_LTseg11_joint: origin xyz=0 0 0.0175 rpy=0 0 0 -> xyz=0 0 0.0125 rpy=0 0 0
- joint LTseg11_LTseg12_joint: origin xyz=0 0 0.0175 rpy=0 0 0 -> xyz=0 0 0.0125 rpy=0 0 0
- joint LTseg1_LTseg2_joint: origin xyz=0 0 0.0175 rpy=0 0 0 -> xyz=0 0 0.0125 rpy=0 0 0
- joint LTseg2_LTseg3_joint: origin xyz=0 0 0.0175 rpy=0 0 0 -> xyz=0 0 0.0125 rpy=0 0 0
- joint LTseg3_LTseg4_joint: origin xyz=0 0 0.0175 rpy=0 0 0 -> xyz=0 0 0.0125 rpy=0 0 0
- joint LTseg4_LTseg5_joint: origin xyz=0 0 0.0175 rpy=0 0 0 -> xyz=0 0 0.0125 rpy=0 0 0
- joint LTseg5_LTseg6_joint: origin xyz=0 0 0.0175 rpy=0 0 0 -> xyz=0 0 0.0125 rpy=0 0 0
- joint LTseg6_LTseg7_joint: origin xyz=0 0 0.0175 rpy=0 0 0 -> xyz=0 0 0.0125 rpy=0 0 0
- joint LTseg7_LTseg8_joint: origin xyz=0 0 0.0175 rpy=0 0 0 -> xyz=0 0 0.0125 rpy=0 0 0
- joint LTseg8_LTseg9_joint: origin xyz=0 0 0.0175 rpy=0 0 0 -> xyz=0 0 0.0125 rpy=0 0 0
- joint LTseg9_LTseg10_joint: origin xyz=0 0 0.0175 rpy=0 0 0 -> xyz=0 0 0.0125 rpy=0 0 0
- joint RBseg10_RBseg11_joint: origin xyz=0 0 0.0175 rpy=0 0 0 -> xyz=0 0 0.0125 rpy=0 0 0
- joint RBseg11_RBseg12_joint: origin xyz=0 0 0.0175 rpy=0 0 0 -> xyz=0 0 0.0125 rpy=0 0 0
- joint RBseg1_RBseg2_joint: origin xyz=0 0 0.0175 rpy=0 0 0 -> xyz=0 0 0.0125 rpy=0 0 0
- joint RBseg2_RBseg3_joint: origin xyz=0 0 0.0175 rpy=0 0 0 -> xyz=0 0 0.0125 rpy=0 0 0
- joint RBseg3_RBseg4_joint: origin xyz=0 0 0.0175 rpy=0 0 0 -> xyz=0 0 0.0125 rpy=0 0 0
- joint RBseg4_RBseg5_joint: origin xyz=0 0 0.0175 rpy=0 0 0 -> xyz=0 0 0.0125 rpy=0 0 0
- joint RBseg5_RBseg6_joint: origin xyz=0 0 0.0175 rpy=0 0 0 -> xyz=0 0 0.0125 rpy=0 0 0
- joint RBseg6_RBseg7_joint: origin xyz=0 0 0.0175 rpy=0 0 0 -> xyz=0 0 0.0125 rpy=0 0 0
- joint RBseg7_RBseg8_joint: origin xyz=0 0 0.0175 rpy=0 0 0 -> xyz=0 0 0.0125 rpy=0 0 0
- joint RBseg8_RBseg9_joint: origin xyz=0 0 0.0175 rpy=0 0 0 -> xyz=0 0 0.0125 rpy=0 0 0
- joint RBseg9_RBseg10_joint: origin xyz=0 0 0.0175 rpy=0 0 0 -> xyz=0 0 0.0125 rpy=0 0 0
- joint RTseg10_RTseg11_joint: origin xyz=0 0 0.0175 rpy=0 0 0 -> xyz=0 0 0.0125 rpy=0 0 0
- joint RTseg11_RTseg12_joint: origin xyz=0 0 0.0175 rpy=0 0 0 -> xyz=0 0 0.0125 rpy=0 0 0
- joint RTseg1_RTseg2_joint: origin xyz=0 0 0.0175 rpy=0 0 0 -> xyz=0 0 0.0125 rpy=0 0 0
- joint RTseg2_RTseg3_joint: origin xyz=0 0 0.0175 rpy=0 0 0 -> xyz=0 0 0.0125 rpy=0 0 0
- joint RTseg3_RTseg4_joint: origin xyz=0 0 0.0175 rpy=0 0 0 -> xyz=0 0 0.0125 rpy=0 0 0
- joint RTseg4_RTseg5_joint: origin xyz=0 0 0.0175 rpy=0 0 0 -> xyz=0 0 0.0125 rpy=0 0 0
- joint RTseg5_RTseg6_joint: origin xyz=0 0 0.0175 rpy=0 0 0 -> xyz=0 0 0.0125 rpy=0 0 0
- joint RTseg6_RTseg7_joint: origin xyz=0 0 0.0175 rpy=0 0 0 -> xyz=0 0 0.0125 rpy=0 0 0
- joint RTseg7_RTseg8_joint: origin xyz=0 0 0.0175 rpy=0 0 0 -> xyz=0 0 0.0125 rpy=0 0 0
- joint RTseg8_RTseg9_joint: origin xyz=0 0 0.0175 rpy=0 0 0 -> xyz=0 0 0.0125 rpy=0 0 0
- joint RTseg9_RTseg10_joint: origin xyz=0 0 0.0175 rpy=0 0 0 -> xyz=0 0 0.0125 rpy=0 0 0
- joint Rev1: origin xyz=0.0 0.0 0.025 rpy=0 0 0 -> xyz=0.0 0.0 0.05 rpy=0 0 0
- joint Rev2: origin xyz=-2.1e-05 0.004903 0.025 rpy=0 0 0 -> xyz=-4.2e-05 0.009807 0.05 rpy=0 0 0
- joint Rev3: origin xyz=0.0 0.0 0.15 rpy=0 0 0 -> xyz=0.0 0.0 0.3 rpy=0 0 0
- joint Rev4: origin xyz=3.3e-05 0.0 0.125 rpy=0 0 0 -> xyz=6.6e-05 0.0 0.25 rpy=0 0 0
- joint palm_arm_joint: origin xyz=0.0 0 0.12 rpy=0 0 0 -> xyz=0.0 0 0.15 rpy=0 0 0

File: urdf/macros2.xacro (robot description, xacro)
@@ -47,5 +47,5 @@
 		<limit effort="${fingerForce}" lower="-0.25" upper="0.25" velocity="0.001"/>
 		<dynamics damping="0.05" friction="0.0"/>
-		<origin xyz="0 0 ${length+0.005}" rpy="0 0 0"/>
+		<origin xyz="0 0 ${length}" rpy="0 0 0"/>
 		<parent link="${seg1}"/>
 		<child link="${seg2}"/>

File: urdf/mainDesign.xacro (robot description, xacro)
@@ -32,5 +32,5 @@
     <parent link="Link4_1"/>
     <child link="palm"/>
-	<origin xyz="0.0 0 0.12" rpy="0 0 0"/>
+	<origin xyz="0.0 0 0.15" rpy="0 0 0"/>
 </joint>
 <finger name="LT">

File: urdf/output.xacro (robot description, xacro)
@@ -29,5 +29,5 @@
     <parent link="Link4_1" />
     <child link="palm" />
-	<origin rpy="0 0 0" xyz="0.0 0 0.12" />
+	<origin rpy="0 0 0" xyz="0.0 0 0.15" />
 </joint>
 <gazebo>
