Commit message: Working plugin with param server

File: scripts/output.xacro (robot description, xacro)
@@ -32,7 +32,10 @@
 </joint>
 <gazebo>
-  <plugin filename="libgazebo_ros_control.so" name="gazebo_ros_control">
-	<robotNamespace />
-  </plugin>
+  	<plugin filename="libgazebo_ros_control.so" name="gazebo_ros_control">
+		<robotNamespace />
+  	</plugin>
+ 	<plugin filename="libmain_description.so" name="main_description">
+		<kConstant> 0.4 </kConstant>
+	</plugin>
 </gazebo>
 </robot>

File: urdf/description_log.urdf (robot description, URDF)
Before this commit: robot Design, 55 links, 54 joints
Joints:
- joint LBseg10_LBseg11_joint: limit lower=-0.25 upper=0.25 effort=0.680555555556 velocity=0.001 -> lower=-2 upper=2 effort=0.680555555556 velocity=0.001
- joint LBseg11_LBseg12_joint: limit lower=-0.25 upper=0.25 effort=0.586805555556 velocity=0.001 -> lower=-2 upper=2 effort=0.586805555556 velocity=0.001
- joint LBseg1_LBseg2_joint: limit lower=-0.25 upper=0.25 effort=1.83680555556 velocity=0.001 -> lower=-2 upper=2 effort=1.83680555556 velocity=0.001
- joint LBseg2_LBseg3_joint: limit lower=-0.25 upper=0.25 effort=1.68055555556 velocity=0.001 -> lower=-2 upper=2 effort=1.68055555556 velocity=0.001
- joint LBseg3_LBseg4_joint: limit lower=-0.25 upper=0.25 effort=1.53125 velocity=0.001 -> lower=-2 upper=2 effort=1.53125 velocity=0.001
- joint LBseg4_LBseg5_joint: limit lower=-0.25 upper=0.25 effort=1.38888888889 velocity=0.001 -> lower=-2 upper=2 effort=1.38888888889 velocity=0.001
- joint LBseg5_LBseg6_joint: limit lower=-0.25 upper=0.25 effort=1.25347222222 velocity=0.001 -> lower=-2 upper=2 effort=1.25347222222 velocity=0.001
- joint LBseg6_LBseg7_joint: limit lower=-0.25 upper=0.25 effort=1.125 velocity=0.001 -> lower=-2 upper=2 effort=1.125 velocity=0.001
- joint LBseg7_LBseg8_joint: limit lower=-0.25 upper=0.25 effort=1.00347222222 velocity=0.001 -> lower=-2 upper=2 effort=1.00347222222 velocity=0.001
- joint LBseg8_LBseg9_joint: limit lower=-0.25 upper=0.25 effort=0.888888888889 velocity=0.001 -> lower=-2 upper=2 effort=0.888888888889 velocity=0.001
- joint LBseg9_LBseg10_joint: limit lower=-0.25 upper=0.25 effort=0.78125 velocity=0.001 -> lower=-2 upper=2 effort=0.78125 velocity=0.001
- joint LTseg10_LTseg11_joint: limit lower=-0.25 upper=0.25 effort=0.680555555556 velocity=0.001 -> lower=-2 upper=2 effort=0.680555555556 velocity=0.001
- joint LTseg11_LTseg12_joint: limit lower=-0.25 upper=0.25 effort=0.586805555556 velocity=0.001 -> lower=-2 upper=2 effort=0.586805555556 velocity=0.001
- joint LTseg1_LTseg2_joint: limit lower=-0.25 upper=0.25 effort=1.83680555556 velocity=0.001 -> lower=-2 upper=2 effort=1.83680555556 velocity=0.001
- joint LTseg2_LTseg3_joint: limit lower=-0.25 upper=0.25 effort=1.68055555556 velocity=0.001 -> lower=-2 upper=2 effort=1.68055555556 velocity=0.001
- joint LTseg3_LTseg4_joint: limit lower=-0.25 upper=0.25 effort=1.53125 velocity=0.001 -> lower=-2 upper=2 effort=1.53125 velocity=0.001
- joint LTseg4_LTseg5_joint: limit lower=-0.25 upper=0.25 effort=1.38888888889 velocity=0.001 -> lower=-2 upper=2 effort=1.38888888889 velocity=0.001
- joint LTseg5_LTseg6_joint: limit lower=-0.25 upper=0.25 effort=1.25347222222 velocity=0.001 -> lower=-2 upper=2 effort=1.25347222222 velocity=0.001
- joint LTseg6_LTseg7_joint: limit lower=-0.25 upper=0.25 effort=1.125 velocity=0.001 -> lower=-2 upper=2 effort=1.125 velocity=0.001
- joint LTseg7_LTseg8_joint: limit lower=-0.25 upper=0.25 effort=1.00347222222 velocity=0.001 -> lower=-2 upper=2 effort=1.00347222222 velocity=0.001
- joint LTseg8_LTseg9_joint: limit lower=-0.25 upper=0.25 effort=0.888888888889 velocity=0.001 -> lower=-2 upper=2 effort=0.888888888889 velocity=0.001
- joint LTseg9_LTseg10_joint: limit lower=-0.25 upper=0.25 effort=0.78125 velocity=0.001 -> lower=-2 upper=2 effort=0.78125 velocity=0.001
- joint RBseg10_RBseg11_joint: limit lower=-0.25 upper=0.25 effort=0.680555555556 velocity=0.001 -> lower=-2 upper=2 effort=0.680555555556 velocity=0.001
- joint RBseg11_RBseg12_joint: limit lower=-0.25 upper=0.25 effort=0.586805555556 velocity=0.001 -> lower=-2 upper=2 effort=0.586805555556 velocity=0.001
- joint RBseg1_RBseg2_joint: limit lower=-0.25 upper=0.25 effort=1.83680555556 velocity=0.001 -> lower=-2 upper=2 effort=1.83680555556 velocity=0.001
- joint RBseg2_RBseg3_joint: limit lower=-0.25 upper=0.25 effort=1.68055555556 velocity=0.001 -> lower=-2 upper=2 effort=1.68055555556 velocity=0.001
- joint RBseg3_RBseg4_joint: limit lower=-0.25 upper=0.25 effort=1.53125 velocity=0.001 -> lower=-2 upper=2 effort=1.53125 velocity=0.001
- joint RBseg4_RBseg5_joint: limit lower=-0.25 upper=0.25 effort=1.38888888889 velocity=0.001 -> lower=-2 upper=2 effort=1.38888888889 velocity=0.001
- joint RBseg5_RBseg6_joint: limit lower=-0.25 upper=0.25 effort=1.25347222222 velocity=0.001 -> lower=-2 upper=2 effort=1.25347222222 velocity=0.001
- joint RBseg6_RBseg7_joint: limit lower=-0.25 upper=0.25 effort=1.125 velocity=0.001 -> lower=-2 upper=2 effort=1.125 velocity=0.001
- joint RBseg7_RBseg8_joint: limit lower=-0.25 upper=0.25 effort=1.00347222222 velocity=0.001 -> lower=-2 upper=2 effort=1.00347222222 velocity=0.001
- joint RBseg8_RBseg9_joint: limit lower=-0.25 upper=0.25 effort=0.888888888889 velocity=0.001 -> lower=-2 upper=2 effort=0.888888888889 velocity=0.001
- joint RBseg9_RBseg10_joint: limit lower=-0.25 upper=0.25 effort=0.78125 velocity=0.001 -> lower=-2 upper=2 effort=0.78125 velocity=0.001
- joint RTseg10_RTseg11_joint: limit lower=-0.25 upper=0.25 effort=0.680555555556 velocity=0.001 -> lower=-2 upper=2 effort=0.680555555556 velocity=0.001
- joint RTseg11_RTseg12_joint: limit lower=-0.25 upper=0.25 effort=0.586805555556 velocity=0.001 -> lower=-2 upper=2 effort=0.586805555556 velocity=0.001
- joint RTseg1_RTseg2_joint: limit lower=-0.25 upper=0.25 effort=1.83680555556 velocity=0.001 -> lower=-2 upper=2 effort=1.83680555556 velocity=0.001
- joint RTseg2_RTseg3_joint: limit lower=-0.25 upper=0.25 effort=1.68055555556 velocity=0.001 -> lower=-2 upper=2 effort=1.68055555556 velocity=0.001
- joint RTseg3_RTseg4_joint: limit lower=-0.25 upper=0.25 effort=1.53125 velocity=0.001 -> lower=-2 upper=2 effort=1.53125 velocity=0.001
- joint RTseg4_RTseg5_joint: limit lower=-0.25 upper=0.25 effort=1.38888888889 velocity=0.001 -> lower=-2 upper=2 effort=1.38888888889 velocity=0.001
- joint RTseg5_RTseg6_joint: limit lower=-0.25 upper=0.25 effort=1.25347222222 velocity=0.001 -> lower=-2 upper=2 effort=1.25347222222 velocity=0.001
- joint RTseg6_RTseg7_joint: limit lower=-0.25 upper=0.25 effort=1.125 velocity=0.001 -> lower=-2 upper=2 effort=1.125 velocity=0.001
- joint RTseg7_RTseg8_joint: limit lower=-0.25 upper=0.25 effort=1.00347222222 velocity=0.001 -> lower=-2 upper=2 effort=1.00347222222 velocity=0.001
- joint RTseg8_RTseg9_joint: limit lower=-0.25 upper=0.25 effort=0.888888888889 velocity=0.001 -> lower=-2 upper=2 effort=0.888888888889 velocity=0.001
- joint RTseg9_RTseg10_joint: limit lower=-0.25 upper=0.25 effort=0.78125 velocity=0.001 -> lower=-2 upper=2 effort=0.78125 velocity=0.001
- joint palm_LBseg1_joint: limit lower=-0.1 upper=0.1 effort=2.0 velocity=0.0001 -> lower=-0.0 upper=0.0 effort=2.0 velocity=0.0001; origin xyz=-0.05 0.05 0 rpy=-0 0 0 -> xyz=-0.04 0.04 0.03 rpy=-0.3 0 0
- joint palm_LTseg1_joint: limit lower=-0.1 upper=0.1 effort=2.0 velocity=0.0001 -> lower=-0.0 upper=0.0 effort=2.0 velocity=0.0001; origin xyz=0.05 0.05 0 rpy=-0 0 0 -> xyz=0.04 0.04 0.03 rpy=-0.3 0 0
- joint palm_RBseg1_joint: limit lower=-0.1 upper=0.1 effort=2.0 velocity=0.0001 -> lower=-0.0 upper=0.0 effort=2.0 velocity=0.0001; origin xyz=-0.05 -0.05 0 rpy=-0 0 3.14159 -> xyz=-0.04 -0.04 0.03 rpy=-0.3 0 3.14159
- joint palm_RTseg1_joint: limit lower=-0.1 upper=0.1 effort=2.0 velocity=0.0001 -> lower=-0.0 upper=0.0 effort=2.0 velocity=0.0001; origin xyz=0.05 -0.05 0 rpy=-0 0 3.14159 -> xyz=0.04 -0.04 0.03 rpy=-0.3 0 3.14159

File: urdf/macros2.xacro (robot description, xacro)
@@ -36,4 +36,5 @@
 	</link>
 	<gazebo reference="${name}">
+		<!--plugin name='main_description' filename='libmain_description.so'/>-->
 		<mu1>20000</mu1>
 		<mu2>20000</mu2>
@@ -45,5 +46,5 @@
 	<joint name="${seg1}_${seg2}_joint" type="revolute">
 		<axis xyz="1 0 0"/>
-		<limit effort="${force}" lower="-0.25" upper="0.25" velocity="0.001"/>
+		<limit effort="${force}" lower="-2" upper="2" velocity="0.001"/>
 		<dynamics damping="0.05" friction="0.0"/>
 		<origin xyz="0 0 ${length}" rpy="0 0 0"/>
@@ -58,5 +59,5 @@
 	<joint name="${seg1}_${seg2}_joint" type="revolute">
 		<axis xyz="1 0 0"/>
-		<limit effort="${force}" lower="-0.1" upper="0.1" velocity="0.0001"/>
+		<limit effort="${force}" lower="-0.0" upper="0.0" velocity="0.0001"/>
 		<!--<dynamics damping="0.05" friction="0.0"/>-->
 		<origin xyz="${offset}" rpy="${rotation}"/>

File: urdf/mainDesign.xacro (robot description, xacro)
@@ -39,5 +39,5 @@
 	<length value="0.15"/>
 	<geometry base = "0.02 0.02" tip = "0.01 0.01"/>
-	<origin xyz="0.05 0.05 0" rpy="-0 0 0"/>
+	<origin xyz="0.04 0.04 0.03" rpy="-0.3 0 0"/>
 	<force value="2"/>
 </finger>
@@ -47,5 +47,5 @@
 	<length value="0.15"/>
 	<geometry base = "0.02 0.02" tip = "0.01 0.01"/>
-	<origin xyz="0.05 -0.05 0" rpy="-0 0 3.14159"/>
+	<origin xyz="0.04 -0.04 0.03" rpy="-0.3 0 3.14159"/>
 	<force value="2"/>
 </finger>
@@ -55,5 +55,5 @@
 	<length value="0.15"/>
 	<geometry base = "0.02 0.02" tip = "0.01 0.01"/>
-	<origin xyz="-0.05 0.05 0" rpy="-0 0 0"/>
+	<origin xyz="-0.04 0.04 0.03" rpy="-0.3 0 0"/>
 	<force value="2"/>
 </finger>
@@ -63,11 +63,14 @@
 	<geometry base = "0.02 0.02" tip = "0.01 0.01"/>
 	<length value="0.15"/>
-	<origin xyz="-0.05 -0.05 0" rpy="-0 0 3.14159"/>
+	<origin xyz="-0.04 -0.04 0.03" rpy="-0.3 0 3.14159"/>
 	<force value="2"/>
 </finger>
 <gazebo>
-  <plugin filename="libgazebo_ros_control.so" name="gazebo_ros_control">
-	<robotNamespace></robotNamespace>
-  </plugin>
+  	<plugin filename="libgazebo_ros_control.so" name="gazebo_ros_control">
+		<robotNamespace></robotNamespace>
+  	</plugin>
+ 	<plugin name='main_description' filename='libmain_description.so'>
+		<kConstant> 0.4 </kConstant>
+	</plugin>
 </gazebo>
 </robot>

File: urdf/output.xacro (robot description, xacro)
@@ -32,11 +32,14 @@
 </joint>
 <gazebo>
-  <plugin filename="libgazebo_ros_control.so" name="gazebo_ros_control">
-	<robotNamespace />
-  </plugin>
+  	<plugin filename="libgazebo_ros_control.so" name="gazebo_ros_control">
+		<robotNamespace />
+  	</plugin>
+ 	<plugin filename="libmain_description.so" name="main_description">
+		<kConstant> 0.4 </kConstant>
+	</plugin>
 </gazebo>
  <!--  MACROS FOR FINGER: LT-->
 <xacro:seg name= "LTseg1" length = "0.0125" height = "0.02" width = "0.02" />
-<xacro:seg_joint_offset seg1= "palm" seg2="LTseg1" length="0.0125" offset="0.05 0.05 0" rotation="-0 0 0" force="2.0" />
+<xacro:seg_joint_offset seg1= "palm" seg2="LTseg1" length="0.0125" offset="0.04 0.04 0.03" rotation="-0.3 0 0" force="2.0" />
 <xacro:seg_trans seg1="palm" seg2="LTseg1"/>
 <xacro:segment name= "LTseg2" parent="LTseg1" length="0.0125" height="0.0191666666667" width = "0.0191666666667" force = "1.83680555556" />
@@ -53,5 +56,5 @@
  <!--  MACROS FOR FINGER: RT-->
 <xacro:seg name= "RTseg1" length = "0.0125" height = "0.02" width = "0.02" />
-<xacro:seg_joint_offset seg1= "palm" seg2="RTseg1" length="0.0125" offset="0.05 -0.05 0" rotation="-0 0 3.14159" force="2.0" />
+<xacro:seg_joint_offset seg1= "palm" seg2="RTseg1" length="0.0125" offset="0.04 -0.04 0.03" rotation="-0.3 0 3.14159" force="2.0" />
 <xacro:seg_trans seg1="palm" seg2="RTseg1"/>
 <xacro:segment name= "RTseg2" parent="RTseg1" length="0.0125" height="0.0191666666667" width = "0.0191666666667" force = "1.83680555556" />
@@ -68,5 +71,5 @@
  <!--  MACROS FOR FINGER: LB-->
 <xacro:seg name= "LBseg1" length = "0.0125" height = "0.02" width = "0.02" />
-<xacro:seg_joint_offset seg1= "palm" seg2="LBseg1" length="0.0125" offset="-0.05 0.05 0" rotation="-0 0 0" force="2.0" />
+<xacro:seg_joint_offset seg1= "palm" seg2="LBseg1" length="0.0125" offset="-0.04 0.04 0.03" rotation="-0.3 0 0" force="2.0" />
 <xacro:seg_trans seg1="palm" seg2="LBseg1"/>
 <xacro:segment name= "LBseg2" parent="LBseg1" length="0.0125" height="0.0191666666667" width = "0.0191666666667" force = "1.83680555556" />
@@ -83,5 +86,5 @@
  <!--  MACROS FOR FINGER: RB-->
 <xacro:seg name= "RBseg1" length = "0.0125" height = "0.02" width = "0.02" />
-<xacro:seg_joint_offset seg1= "palm" seg2="RBseg1" length="0.0125" offset="-0.05 -0.05 0" rotation="-0 0 3.14159" force="2.0" />
+<xacro:seg_joint_offset seg1= "palm" seg2="RBseg1" length="0.0125" offset="-0.04 -0.04 0.03" rotation="-0.3 0 3.14159" force="2.0" />
 <xacro:seg_trans seg1="palm" seg2="RBseg1"/>
 <xacro:segment name= "RBseg2" parent="RBseg1" length="0.0125" height="0.0191666666667" width = "0.0191666666667" force = "1.83680555556" />

Commit message: Major gripper visualiser update

File: scripts/output.xacro (robot description, xacro)
@@ -39,5 +39,8 @@
 	</plugin>
 	<plugin filename="libjoint_controller_plugin.so" name="joint_controller_plugin">
-		<jointNamesParam> "/arm_joints/joints" </jointNamesParam>
+		<jointNamesParam> arm_controller/ </jointNamesParam>
+	</plugin>
+	<plugin filename="libjoint_force_visualiser_plugin.so" name="joint_force_visualier_plugin">
+		<robotNamespace />
 	</plugin>
 </gazebo>

File: urdf/arm.xacro (robot description, xacro)
@@ -5,5 +5,5 @@
 <xacro:include filename="$(find main_description)/urdf/Design.trans" />
 <!--  PROPERTIES  -->
-<xacro:property name="strength" value="1000"/>
+<xacro:property name="strength" value="10000"/>
 <xacro:property name="speed" value = "0.01"/>
 <xacro:property name="damping" value = "0"/>

File: urdf/description_log.urdf (robot description, URDF)
Before this commit: robot Design, 55 links, 54 joints
Joints:
- joint Rev1: limit lower=-6.283185 upper=6.283185 effort=1000 velocity=0.01 -> lower=-6.283185 upper=6.283185 effort=10000 velocity=0.01
- joint Rev2: limit lower=-1.396263 upper=1.396263 effort=1000 velocity=0.01 -> lower=-1.396263 upper=1.396263 effort=10000 velocity=0.01
- joint Rev3: limit lower=-2.792527 upper=2.792527 effort=1000 velocity=0.01 -> lower=-2.792527 upper=2.792527 effort=10000 velocity=0.01
- joint Rev4: limit lower=-2.617994 upper=2.617994 effort=1000 velocity=0.01 -> lower=-2.617994 upper=2.617994 effort=10000 velocity=0.01

File: urdf/macros2.xacro (robot description, xacro)
@@ -47,5 +47,5 @@
 		<axis xyz="1 0 0"/>
 		<limit effort="${force}" lower="-2" upper="2" velocity="0.001"/>
-		<dynamics damping="0.05" friction="0.0"/>
+		<dynamics damping="0.02" friction="0.0"/>
 		<origin xyz="0 0 ${length}" rpy="0 0 0"/>
 		<parent link="${seg1}"/>

File: urdf/mainDesign.xacro (robot description, xacro)
@@ -74,5 +74,8 @@
 	</plugin>
 	<plugin name="joint_controller_plugin" filename ="libjoint_controller_plugin.so">
-		<jointNamesParam> "/arm_joints/joints" </jointNamesParam>
+		<jointNamesParam> arm_controller/ </jointNamesParam>
+	</plugin>
+	<plugin name="joint_force_visualier_plugin" filename="libjoint_force_visualiser_plugin.so">
+		<robotNamespace></robotNamespace>
 	</plugin>
 </gazebo>

File: urdf/output.xacro (robot description, xacro)
@@ -39,5 +39,8 @@
 	</plugin>
 	<plugin filename="libjoint_controller_plugin.so" name="joint_controller_plugin">
-		<jointNamesParam> "/arm_joints/joints" </jointNamesParam>
+		<jointNamesParam> arm_controller/ </jointNamesParam>
+	</plugin>
+	<plugin filename="libjoint_force_visualiser_plugin.so" name="joint_force_visualier_plugin">
+		<robotNamespace />
 	</plugin>
 </gazebo>
